File: blahajmacro.kicad_pcb (KiCad board)
At the start: 2 copper layers, 90.5 x 63 mm, 16 parts, among them J1 OLED_128x32, SW1 RotaryEncoder_Switch, SW2 RotaryEncoder_Switch, U1 Seeed Studio XIAO SAMD21

Commit message: Completed pcb
Parts:
- removed the G*** at (113.4, 54.4)
- added G***: LOGO, LOGO, B.Cu at (139.6, 39.0)
- added G***: LOGO, LOGO, B.Cu at (149.4, 25.2)
- added G***: LOGO, LOGO, B.Cu at (101.5, 41.8)
- added G***: LOGO, LOGO, B.Cu at (81.0, 71.5)
- added G***: LOGO, LOGO, B.Cu at (116.6, 54.2)
- added G***: LOGO, LOGO, B.Cu at (143.3, 65.0)
- D1, D2, D3, D4, D5, D6: moved to B.Cu
- U1: value Seeed Studio XIAO SAMD21 -> MCU_Seeed_XIAO_RP2040; moved to B.Cu
- moved G*** 36.2 mm to (117.9, 75.5)
- moved S3 1.86 mm to (125.6, 50.4)
- moved S1 1.86 mm to (87.5, 50.4)
- moved S2 1.86 mm to (106.5, 50.4)
- moved S4 1.86 mm to (144.6, 50.4)
- moved U1 1.16 mm to (83.8, 33.3), turned to 180 degrees
Connections:
- J1 pad 2: +5V -> +3V3
- U1 pad 1: ROW3 -> ROW1
- U1 pad 12: unconnected-(U1-3V3-Pad12)_1 -> +3V3
- U1 pad 14: +5V -> unconnected-(U1-5V-Pad14)
- U1 pad 3: ROW1 -> ROW3
- U1 pad 4: COL2 -> COL1
- U1 pad 7: COL1 -> COL2
- U1 pad 8: ROTA1 -> ROTB1
- U1 pad 9: ROTB1 -> ROTA1
Routing:
- net ROW1: track 77.5 -> 174.8 mm
- net +3V3: track 0.00 -> 67.2 mm
- net ROW2: track 101.0 -> 156.1 mm
- net +5V: track 40.0 -> 0.00 mm
- net SDA: track 63.2 -> 34.7 mm
- net SCL: track 58.9 -> 34.7 mm
- net COL2: track 147.6 -> 124.6 mm
- net ROTB1: track 49.9 -> 29.5 mm
- net COL1: track 71.8 -> 90.8 mm
- net ROTB2: track 88.7 -> 107.2 mm
- net ROTA2: track 97.2 -> 115.6 mm
- net ROW3: track 122.2 -> 136.5 mm
- net Net-(D4-A): track 40.2 -> 46.8 mm
- net GND: track 180.8 -> 185.8 mm
- net Net-(D1-A): track 25.3 -> 23.4 mm
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