File: blahajmacro.kicad_sch (KiCad schematic)
At the start: 14 parts, among them J1 OLED_128x32, SW1 RotaryEncoder_Switch, SW2 RotaryEncoder_Switch, U1 Seeed Studio XIAO SAMD21

Commit message: Completed pcb
Parts:
- removed U1: Seeed Studio XIAO SAMD21, ScottoKeebs_MCU:Seeed_XIAO_RP2040, symbol Seeed_Studio_XIAO_Series:Seeed Studio XIAO SAMD21
- added U1: MCU_Seeed_XIAO_RP2040, ScottoKeebs_MCU:Seeed_XIAO_RP2040, symbol ScottoKeebs:MCU_Seeed_XIAO_RP2040
Connections:
- net COL1: now also U1.4 (PA11_A3_D3)
- net COL2: now also U1.7 (PB08_A6_D6_TX)
- net GND: now also U1.13 (GND)
- net ROTA1: now also U1.9 (PA7_A8_D8_SCK)
- net ROTA2: now also U1.11 (PA6_A10_D10_MOSI)
- net ROTB1: now also U1.8 (PB09_A7_D7_RX)
- net ROTB2: now also U1.10 (PA5_A9_D9_MISO)
- net ROW1: now also U1.1 (PA02_A0_D0)
- net ROW2: now also U1.2 (PA4_A1_D1)
- net ROW3: now also U1.3 (PA10_A2_D2)
- net SCL: now also U1.6 (PA9_A5_D5_SCL)
- net SDA: now also U1.5 (PA8_A4_D4_SDA)
- net +5V renamed +3V3
- net +3V3: now also U1.12 (3V3)
- no-connect marks 4 -> 1
